Commit message: working version

File: urdf/udacity_bot.xacro (robot description, xacro)
@@ -40,4 +40,20 @@
     <joint_properties damping="1.0" friction="1.0"/>
   </joint>
+  <joint type="fixed" name="front_caster_joint">
+    <origin xyz="0.15 0 -0.05" rpy="0 0 0"/>
+    <child link="front_caster"/>
+    <parent link="chassis"/>
+    <axis xyz="0 1 0" rpy="0 0 0"/>
+    <limit effort="10000" velocity="1000"/>
+    <joint_properties damping="1.0" friction="1.0"/>
+  </joint>
+  <joint type="fixed" name="back_caster_joint">
+    <origin xyz="-0.15 0 -0.05" rpy="0 0 0"/>
+    <child link="back_caster"/>
+    <parent link="chassis"/>
+    <axis xyz="0 1 0" rpy="0 0 0"/>
+    <limit effort="10000" velocity="1000"/>
+    <joint_properties damping="1.0" friction="1.0"/>
+  </joint>
   <link name='left_wheel'>
     <inertial>
@@ -155,6 +171,8 @@
       </geometry>
     </visual>
-    <collision name='back_caster_collision'>
-      <origin xyz="-0.15 0 -0.05" rpy=" 0 0 0"/>
+  </link>
+  <link name='front_caster'>
+    <collision name='front_caster_collision'>
+      <origin xyz="0 0 0" rpy=" 0 0 0"/>
       <geometry>
         <sphere radius="0.05"/>
@@ -171,12 +189,14 @@
       </surface>
     </collision>
-    <visual name='back_caster_visual'>
-      <origin xyz="-0.15 0 -0.05" rpy=" 0 0 0"/>
-      <geometry>
-        <sphere radius="0.05"/>
-      </geometry>
-    </visual>
-    <collision name='front_caster_collision'>
-      <origin xyz="0.15 0 -0.05" rpy=" 0 0 0"/>
+    <visual name='front_caster_visual'>
+      <origin xyz="0 0 0" rpy=" 0 0 0"/>
+      <geometry>
+        <sphere radius="0.05"/>
+      </geometry>
+    </visual>
+  </link>
+  <link name='back_caster'>
+      <collision name='back_caster_collision'>
+      <origin xyz="0 0 0" rpy=" 0 0 0"/>
       <geometry>
         <sphere radius="0.05"/>
@@ -193,6 +213,6 @@
       </surface>
     </collision>
-    <visual name='front_caster_visual'>
-      <origin xyz="0.15 0 -0.05" rpy=" 0 0 0"/>
+    <visual name='back_caster_visual'>
+      <origin xyz="0 0 0" rpy=" 0 0 0"/>
       <geometry>
         <sphere radius="0.05"/>
